Commit message: urdf with slider installed

File: franka_description/robots/common/franka_arm.xacro (robot description, xacro)
@@ -20,9 +20,9 @@
     <xacro:link_with_sc name="link1" gazebo="${gazebo}">
       <self_collision_geometries>
-        <xacro:collision_capsule xyz="0 0 -191.5e-3" radius="${0.06+safety_distance}" length="0.283" />
+        <xacro:collision_capsule xyz="0 0 0" radius="${0.06+safety_distance}" length="0.1" />
       </self_collision_geometries>
     </xacro:link_with_sc>
-    <joint name="${arm_id}_joint1" type="revolute">
-      <origin rpy="0 0 0" xyz="0 0 0.333" />
+    <joint name="${arm_id}_joint1" type="prismatic">
+      <origin rpy="${pi/2} 0 0" xyz="-0.39 1.1 0.6" />
       <parent link="${arm_id}_link0" />
       <child link="${arm_id}_link1" />
@@ -33,22 +33,20 @@
     <xacro:link_with_sc name="link2" gazebo="${gazebo}">
       <self_collision_geometries>
-        <xacro:collision_capsule xyz="0 0 0" radius="${0.06+safety_distance}" length="0.12" />
+        <xacro:collision_capsule xyz="0 0 -191.5e-3" radius="${0.06+safety_distance}" length="0.283" />
       </self_collision_geometries>
     </xacro:link_with_sc>
-    <joint name="${arm_id}_joint2" type="revolute">
-      <origin rpy="${-pi/2} 0 0" xyz="0 0 0" />
+    <joint name="${arm_id}_joint2" type="fixed">
+      <origin rpy="${-pi/2} 0 0" xyz="-0.074 0.036 -0.145 " />
       <parent link="${arm_id}_link1" />
       <child link="${arm_id}_link2" />
-      <axis xyz="0 0 1" />
       <xacro:franka-limits name="joint2" config="${joint_limits}" />
-      <dynamics D="1" K="7000" damping="0.003" friction="0.0" mu_coulomb="0" mu_viscous="16" />
     </joint>
     <xacro:link_with_sc name="link3" gazebo="${gazebo}">
       <self_collision_geometries>
-        <xacro:collision_capsule xyz="0 0 -0.145" radius="${0.06+safety_distance}" length="0.15" />
+        <xacro:collision_capsule xyz="0 0 -191.5e-3" radius="${0.06+safety_distance}" length="0.283" />
       </self_collision_geometries>
     </xacro:link_with_sc>
     <joint name="${arm_id}_joint3" type="revolute">
-      <origin rpy="${pi/2} 0 0" xyz="0 -0.316 0" />
+      <origin rpy="0 0 0" xyz="0 0 0.333" />
       <parent link="${arm_id}_link2" />
       <child link="${arm_id}_link3" />
@@ -60,8 +58,8 @@
       <self_collision_geometries>
         <xacro:collision_capsule xyz="0 0 0" radius="${0.06+safety_distance}" length="0.12" />
-     </self_collision_geometries>
+      </self_collision_geometries>
     </xacro:link_with_sc>
     <joint name="${arm_id}_joint4" type="revolute">
-      <origin rpy="${pi/2} 0 0" xyz="0.0825 0 0" />
+      <origin rpy="${-pi/2} 0 0" xyz="0 0 0" />
       <parent link="${arm_id}_link3" />
       <child link="${arm_id}_link4" />
@@ -72,10 +70,9 @@
     <xacro:link_with_sc name="link5" gazebo="${gazebo}">
       <self_collision_geometries>
-        <xacro:collision_capsule xyz="0 0 -0.26"    radius="${0.060+safety_distance}" length="0.10" />
-        <xacro:collision_capsule xyz="0 0.08 -0.13" radius="${0.025+safety_distance}" length="0.14" />
+        <xacro:collision_capsule xyz="0 0 -0.145" radius="${0.06+safety_distance}" length="0.15" />
       </self_collision_geometries>
     </xacro:link_with_sc>
     <joint name="${arm_id}_joint5" type="revolute">
-      <origin rpy="${-pi/2} 0 0" xyz="-0.0825 0.384 0" />
+      <origin rpy="${pi/2} 0 0" xyz="0 -0.316 0" />
       <parent link="${arm_id}_link4" />
       <child link="${arm_id}_link5" />
@@ -86,9 +83,9 @@
     <xacro:link_with_sc name="link6" gazebo="${gazebo}">
       <self_collision_geometries>
-        <xacro:collision_capsule xyz="0 0 -0.03" radius="${0.05+safety_distance}" length="0.08" />
-      </self_collision_geometries>
+        <xacro:collision_capsule xyz="0 0 0" radius="${0.06+safety_distance}" length="0.12" />
+     </self_collision_geometries>
     </xacro:link_with_sc>
     <joint name="${arm_id}_joint6" type="revolute">
-      <origin rpy="${pi/2} 0 0" xyz="0 0 0" />
+      <origin rpy="${pi/2} 0 0" xyz="0.0825 0 0" />
       <parent link="${arm_id}_link5" />
       <child link="${arm_id}_link6" />
@@ -97,5 +94,32 @@
       <dynamics D="1" K="7000" damping="0.003" friction="0.0" mu_coulomb="0" mu_viscous="16" />
     </joint>
-    <xacro:link_with_sc name="link7" gazebo="${gazebo}" rpy="0 0 ${pi/4}">
+    <xacro:link_with_sc name="link7" gazebo="${gazebo}">
+      <self_collision_geometries>
+        <xacro:collision_capsule xyz="0 0 -0.26"    radius="${0.060+safety_distance}" length="0.10" />
+        <xacro:collision_capsule xyz="0 0.08 -0.13" radius="${0.025+safety_distance}" length="0.14" />
+      </self_collision_geometries>
+    </xacro:link_with_sc>
+    <joint name="${arm_id}_joint7" type="revolute">
+      <origin rpy="${-pi/2} 0 0" xyz="-0.0825 0.384 0" />
+      <parent link="${arm_id}_link6" />
+      <child link="${arm_id}_link7" />
+      <axis xyz="0 0 1" />
+      <xacro:franka-limits name="joint7" config="${joint_limits}" />
+      <dynamics D="1" K="7000" damping="0.003" friction="0.0" mu_coulomb="0" mu_viscous="16" />
+    </joint>
+    <xacro:link_with_sc name="link8" gazebo="${gazebo}">
+      <self_collision_geometries>
+        <xacro:collision_capsule xyz="0 0 -0.03" radius="${0.05+safety_distance}" length="0.08" />
+      </self_collision_geometries>
+    </xacro:link_with_sc>
+    <joint name="${arm_id}_joint8" type="revolute">
+      <origin rpy="${pi/2} 0 0" xyz="0 0 0" />
+      <parent link="${arm_id}_link7" />
+      <child link="${arm_id}_link8" />
+      <axis xyz="0 0 1" />
+      <xacro:franka-limits name="joint8" config="${joint_limits}" />
+      <dynamics D="1" K="7000" damping="0.003" friction="0.0" mu_coulomb="0" mu_viscous="16" />
+    </joint>
+    <xacro:link_with_sc name="link9" gazebo="${gazebo}" rpy="0 0 ${pi/4}">
       <self_collision_geometries>
         <xacro:collision_capsule xyz="0 0 0.01" direction="z" radius="${0.04+safety_distance}" length="0.14" />
@@ -103,17 +127,17 @@
       </self_collision_geometries>
     </xacro:link_with_sc>
-    <joint name="${arm_id}_joint7" type="revolute">
+    <joint name="${arm_id}_joint9" type="revolute">
       <origin rpy="${pi/2} 0 0" xyz="0.088 0 0"/>
-      <parent link="${arm_id}_link6"/>
-      <child link="${arm_id}_link7"/>
+      <parent link="${arm_id}_link8"/>
+      <child link="${arm_id}_link9"/>
       <axis xyz="0 0 1"/>
-      <xacro:franka-limits name="joint7" config="${joint_limits}" />
+      <xacro:franka-limits name="joint9" config="${joint_limits}" />
       <dynamics D="1" K="7000" damping="0.003" friction="0.0" mu_coulomb="0" mu_viscous="16"/>
     </joint>
-    <link name="${arm_id}_link8"/>
-    <joint name="${arm_id}_joint8" type="fixed">
+    <link name="${arm_id}_link10"/>
+    <joint name="${arm_id}_joint10" type="fixed">
       <origin rpy="0 0 0" xyz="0 0 0.107"/>
-      <parent link="${arm_id}_link7"/>
-      <child link="${arm_id}_link8"/>
+      <parent link="${arm_id}_link9"/>
+      <child link="${arm_id}_link10"/>
     </joint>
   </xacro:macro>

File: franka_description/robots/common/franka_robot.xacro (robot description, xacro)
@@ -12,5 +12,5 @@
           tcp_xyz="${tcp_xyz}"
           tcp_rpy="${tcp_rpy}"
-          connected_to="${arm_id}_link8"
+          connected_to="${arm_id}_link10"
           safety_distance="0.03"
           gazebo="${gazebo}"
@@ -31,5 +31,4 @@
       </xacro:if>
       <xacro:gazebo-joint joint="${arm_id}_joint1" transmission="hardware_interface/PositionJointInterface" />
-      <xacro:gazebo-joint joint="${arm_id}_joint2" transmission="hardware_interface/PositionJointInterface" />
       <xacro:gazebo-joint joint="${arm_id}_joint3" transmission="hardware_interface/PositionJointInterface" />
       <xacro:gazebo-joint joint="${arm_id}_joint4" transmission="hardware_interface/PositionJointInterface" />
@@ -37,6 +36,7 @@
       <xacro:gazebo-joint joint="${arm_id}_joint6" transmission="hardware_interface/PositionJointInterface" />
       <xacro:gazebo-joint joint="${arm_id}_joint7" transmission="hardware_interface/PositionJointInterface" />
+      <xacro:gazebo-joint joint="${arm_id}_joint8" transmission="hardware_interface/PositionJointInterface" />
+      <xacro:gazebo-joint joint="${arm_id}_joint9" transmission="hardware_interface/PositionJointInterface" />
       <xacro:gazebo-joint joint="${arm_id}_joint1" transmission="hardware_interface/VelocityJointInterface" />
-      <xacro:gazebo-joint joint="${arm_id}_joint2" transmission="hardware_interface/VelocityJointInterface" />
       <xacro:gazebo-joint joint="${arm_id}_joint3" transmission="hardware_interface/VelocityJointInterface" />
       <xacro:gazebo-joint joint="${arm_id}_joint4" transmission="hardware_interface/VelocityJointInterface" />
@@ -44,6 +44,7 @@
       <xacro:gazebo-joint joint="${arm_id}_joint6" transmission="hardware_interface/VelocityJointInterface" />
       <xacro:gazebo-joint joint="${arm_id}_joint7" transmission="hardware_interface/VelocityJointInterface" />
+      <xacro:gazebo-joint joint="${arm_id}_joint8" transmission="hardware_interface/VelocityJointInterface" />
+      <xacro:gazebo-joint joint="${arm_id}_joint9" transmission="hardware_interface/PositionJointInterface" />
       <xacro:gazebo-joint joint="${arm_id}_joint1" transmission="hardware_interface/EffortJointInterface" />
-      <xacro:gazebo-joint joint="${arm_id}_joint2" transmission="hardware_interface/EffortJointInterface" />
       <xacro:gazebo-joint joint="${arm_id}_joint3" transmission="hardware_interface/EffortJointInterface" />
       <xacro:gazebo-joint joint="${arm_id}_joint4" transmission="hardware_interface/EffortJointInterface" />
@@ -51,8 +52,10 @@
       <xacro:gazebo-joint joint="${arm_id}_joint6" transmission="hardware_interface/EffortJointInterface" />
       <xacro:gazebo-joint joint="${arm_id}_joint7" transmission="hardware_interface/EffortJointInterface" />
+      <xacro:gazebo-joint joint="${arm_id}_joint8" transmission="hardware_interface/EffortJointInterface" />
+      <xacro:gazebo-joint joint="${arm_id}_joint9" transmission="hardware_interface/PositionJointInterface" />
       <xacro:transmission-franka-state arm_id="${arm_id}" />
       <xacro:transmission-franka-model arm_id="${arm_id}"
          root="${arm_id}_joint1"
-         tip="${arm_id}_joint8"
+         tip="${arm_id}_joint9"
        />
       <xacro:if value="${hand}">

File: franka_description/robots/common/utils.xacro (robot description, xacro)
@@ -160,5 +160,4 @@
       <type>franka_hw/FrankaStateInterface</type>
       <joint name="${arm_id}_joint1"><hardwareInterface>franka_hw/FrankaStateInterface</hardwareInterface></joint>
-      <joint name="${arm_id}_joint2"><hardwareInterface>franka_hw/FrankaStateInterface</hardwareInterface></joint>
       <joint name="${arm_id}_joint3"><hardwareInterface>franka_hw/FrankaStateInterface</hardwareInterface></joint>
       <joint name="${arm_id}_joint4"><hardwareInterface>franka_hw/FrankaStateInterface</hardwareInterface></joint>
@@ -166,6 +165,7 @@
       <joint name="${arm_id}_joint6"><hardwareInterface>franka_hw/FrankaStateInterface</hardwareInterface></joint>
       <joint name="${arm_id}_joint7"><hardwareInterface>franka_hw/FrankaStateInterface</hardwareInterface></joint>
+      <joint name="${arm_id}_joint8"><hardwareInterface>franka_hw/FrankaStateInterface</hardwareInterface></joint>
+      <joint name="${arm_id}_joint9"><hardwareInterface>franka_hw/FrankaStateInterface</hardwareInterface></joint>
       <actuator name="${arm_id}_motor1"><hardwareInterface>franka_hw/FrankaStateInterface</hardwareInterface></actuator>
-      <actuator name="${arm_id}_motor2"><hardwareInterface>franka_hw/FrankaStateInterface</hardwareInterface></actuator>
       <actuator name="${arm_id}_motor3"><hardwareInterface>franka_hw/FrankaStateInterface</hardwareInterface></actuator>
       <actuator name="${arm_id}_motor4"><hardwareInterface>franka_hw/FrankaStateInterface</hardwareInterface></actuator>
@@ -173,4 +173,6 @@
       <actuator name="${arm_id}_motor6"><hardwareInterface>franka_hw/FrankaStateInterface</hardwareInterface></actuator>
       <actuator name="${arm_id}_motor7"><hardwareInterface>franka_hw/FrankaStateInterface</hardwareInterface></actuator>
+      <actuator name="${arm_id}_motor8"><hardwareInterface>franka_hw/FrankaStateInterface</hardwareInterface></actuator>
+      <actuator name="${arm_id}_motor9"><hardwareInterface>franka_hw/FrankaStateInterface</hardwareInterface></actuator>
     </transmission>
   </xacro:macro>

Commit message: files with preliminary controller

File: franka_description/robots/common/franka_arm.xacro (robot description, xacro)
@@ -13,9 +13,33 @@
       </joint>
     </xacro:unless>
-    <xacro:link_with_sc name="link0" gazebo="${gazebo}">
+    <xacro:link_with_sc name="link8" gazebo="${gazebo}">
       <self_collision_geometries>
         <xacro:collision_capsule xyz="-0.075 0 0.06" direction="x" radius="${0.06+safety_distance}" length="0.03" />
       </self_collision_geometries>
     </xacro:link_with_sc>
+    <xacro:link_with_sc name="link9" gazebo="${gazebo}">
+      <self_collision_geometries>
+        <xacro:collision_capsule xyz="0 0 0" radius="${0.06+safety_distance}" length="0.1" />
+      </self_collision_geometries>
+    </xacro:link_with_sc>
+    <joint name="${arm_id}_joint8" type="prismatic">
+      <origin rpy="${pi/2} 0 0" xyz="-0.39 1.1 0.6" />
+      <parent link="${arm_id}_link8" />
+      <child link="${arm_id}_link9" />
+      <axis xyz="0 0 1" />
+      <xacro:franka-limits name="joint8" config="${joint_limits}" />
+      <dynamics D="1" K="7000" damping="0.003" friction="0.0" mu_coulomb="0" mu_viscous="16" />
+    </joint>
+    <xacro:link_with_sc name="link0" gazebo="${gazebo}">
+      <self_collision_geometries>
+        <xacro:collision_capsule xyz="0 0 -191.5e-3" radius="${0.06+safety_distance}" length="0.283" />
+      </self_collision_geometries>
+    </xacro:link_with_sc>
+    <joint name="${arm_id}_joint9" type="fixed">
+      <origin rpy="${-pi/2} 0 0" xyz="-0.074 0.036 -0.145 " />
+      <parent link="${arm_id}_link9" />
+      <child link="${arm_id}_link0" />
+      <xacro:franka-limits name="joint9" config="${joint_limits}" />
+    </joint>
     <xacro:link_with_sc name="link1" gazebo="${gazebo}">
       <self_collision_geometries>
@@ -111,9 +135,9 @@
       <dynamics D="1" K="7000" damping="0.003" friction="0.0" mu_coulomb="0" mu_viscous="16"/>
     </joint>
-    <link name="${arm_id}_link8"/>
-    <joint name="${arm_id}_joint8" type="fixed">
+    <link name="${arm_id}_link10"/>
+    <joint name="${arm_id}_joint10" type="fixed">
       <origin rpy="0 0 0" xyz="0 0 0.107"/>
       <parent link="${arm_id}_link7"/>
-      <child link="${arm_id}_link8"/>
+      <child link="${arm_id}_link10"/>
     </joint>
   </xacro:macro>

File: franka_description/robots/common/franka_robot.xacro (robot description, xacro)
@@ -12,5 +12,5 @@
           tcp_xyz="${tcp_xyz}"
           tcp_rpy="${tcp_rpy}"
-          connected_to="${arm_id}_link8"
+          connected_to="${arm_id}_link10"
           safety_distance="0.03"
           gazebo="${gazebo}"
@@ -31,5 +31,4 @@
       </xacro:if>
       <xacro:gazebo-joint joint="${arm_id}_joint1" transmission="hardware_interface/PositionJointInterface" />
-      <xacro:gazebo-joint joint="${arm_id}_joint2" transmission="hardware_interface/PositionJointInterface" />
       <xacro:gazebo-joint joint="${arm_id}_joint3" transmission="hardware_interface/PositionJointInterface" />
       <xacro:gazebo-joint joint="${arm_id}_joint4" transmission="hardware_interface/PositionJointInterface" />
@@ -37,6 +36,6 @@
       <xacro:gazebo-joint joint="${arm_id}_joint6" transmission="hardware_interface/PositionJointInterface" />
       <xacro:gazebo-joint joint="${arm_id}_joint7" transmission="hardware_interface/PositionJointInterface" />
+      <xacro:gazebo-joint joint="${arm_id}_joint8" transmission="hardware_interface/PositionJointInterface" />
       <xacro:gazebo-joint joint="${arm_id}_joint1" transmission="hardware_interface/VelocityJointInterface" />
-      <xacro:gazebo-joint joint="${arm_id}_joint2" transmission="hardware_interface/VelocityJointInterface" />
       <xacro:gazebo-joint joint="${arm_id}_joint3" transmission="hardware_interface/VelocityJointInterface" />
       <xacro:gazebo-joint joint="${arm_id}_joint4" transmission="hardware_interface/VelocityJointInterface" />
@@ -44,6 +43,6 @@
       <xacro:gazebo-joint joint="${arm_id}_joint6" transmission="hardware_interface/VelocityJointInterface" />
       <xacro:gazebo-joint joint="${arm_id}_joint7" transmission="hardware_interface/VelocityJointInterface" />
+      <xacro:gazebo-joint joint="${arm_id}_joint8" transmission="hardware_interface/VelocityJointInterface" />
       <xacro:gazebo-joint joint="${arm_id}_joint1" transmission="hardware_interface/EffortJointInterface" />
-      <xacro:gazebo-joint joint="${arm_id}_joint2" transmission="hardware_interface/EffortJointInterface" />
       <xacro:gazebo-joint joint="${arm_id}_joint3" transmission="hardware_interface/EffortJointInterface" />
       <xacro:gazebo-joint joint="${arm_id}_joint4" transmission="hardware_interface/EffortJointInterface" />
@@ -51,8 +50,9 @@
       <xacro:gazebo-joint joint="${arm_id}_joint6" transmission="hardware_interface/EffortJointInterface" />
       <xacro:gazebo-joint joint="${arm_id}_joint7" transmission="hardware_interface/EffortJointInterface" />
+      <xacro:gazebo-joint joint="${arm_id}_joint8" transmission="hardware_interface/EffortJointInterface" />
       <xacro:transmission-franka-state arm_id="${arm_id}" />
       <xacro:transmission-franka-model arm_id="${arm_id}"
          root="${arm_id}_joint1"
-         tip="${arm_id}_joint8"
+         tip="${arm_id}_joint10"
        />
       <xacro:if value="${hand}">

File: franka_description/robots/common/utils.xacro (robot description, xacro)
@@ -160,5 +160,4 @@
       <type>franka_hw/FrankaStateInterface</type>
       <joint name="${arm_id}_joint1"><hardwareInterface>franka_hw/FrankaStateInterface</hardwareInterface></joint>
-      <joint name="${arm_id}_joint2"><hardwareInterface>franka_hw/FrankaStateInterface</hardwareInterface></joint>
       <joint name="${arm_id}_joint3"><hardwareInterface>franka_hw/FrankaStateInterface</hardwareInterface></joint>
       <joint name="${arm_id}_joint4"><hardwareInterface>franka_hw/FrankaStateInterface</hardwareInterface></joint>
@@ -166,6 +165,6 @@
       <joint name="${arm_id}_joint6"><hardwareInterface>franka_hw/FrankaStateInterface</hardwareInterface></joint>
       <joint name="${arm_id}_joint7"><hardwareInterface>franka_hw/FrankaStateInterface</hardwareInterface></joint>
+      <joint name="${arm_id}_joint8"><hardwareInterface>franka_hw/FrankaStateInterface</hardwareInterface></joint>
       <actuator name="${arm_id}_motor1"><hardwareInterface>franka_hw/FrankaStateInterface</hardwareInterface></actuator>
-      <actuator name="${arm_id}_motor2"><hardwareInterface>franka_hw/FrankaStateInterface</hardwareInterface></actuator>
       <actuator name="${arm_id}_motor3"><hardwareInterface>franka_hw/FrankaStateInterface</hardwareInterface></actuator>
       <actuator name="${arm_id}_motor4"><hardwareInterface>franka_hw/FrankaStateInterface</hardwareInterface></actuator>
@@ -173,4 +172,5 @@
       <actuator name="${arm_id}_motor6"><hardwareInterface>franka_hw/FrankaStateInterface</hardwareInterface></actuator>
       <actuator name="${arm_id}_motor7"><hardwareInterface>franka_hw/FrankaStateInterface</hardwareInterface></actuator>
+      <actuator name="${arm_id}_motor8"><hardwareInterface>franka_hw/FrankaStateInterface</hardwareInterface></actuator>
     </transmission>
   </xacro:macro>
